File: bbq-monitor.sch (KiCad schematic (older format))
At the start: 50 parts, among them J1 Power, J2 USB_B_Mini, Q1 BC847, Q2 BC847, SW1 SW_Push, U1 ESP32-WROOM-32D, U2 TPS62132, U3 USBLC6-2SC6, U4 DHT11, U6 CP2104

Commit message: pcb draft finished
Parts:
- removed C10: 100n, Capacitor_SMD:C_0603_1608Metric, symbol Device:C_Small
- removed R6: 220, Resistor_SMD:R_0603_1608Metric, symbol Device:R_Small
- added R13: 100, Resistor_SMD:R_0603_1608Metric, symbol Device:R_Small
- added R14: 820k, Resistor_SMD:R_0603_1608Metric, symbol Device:R_Small
- added R15: 270k, Resistor_SMD:R_0603_1608Metric, symbol Device:R_Small
- added R4: 220, Resistor_SMD:R_0603_1608Metric, symbol Device:R_Small
- F1: value 3A -> 1A
- H1: renamed from H4; footprint MountingHole:MountingHole_4.3mm_M4_Pad_Via -> MountingHole:MountingHole_3.2mm_M3_Pad_Via
- H2, H3: footprint MountingHole:MountingHole_4.3mm_M4_Pad_Via -> MountingHole:MountingHole_3.2mm_M3_Pad_Via
- H4: renamed from H1; footprint MountingHole:MountingHole_4.3mm_M4_Pad_Via -> MountingHole:MountingHole_3.2mm_M3_Pad_Via
- R2: renamed from R3; value 0 -> 470
- R3: renamed from R4; value 0 -> 470
- gave numbers to parts that had none: 11
- renumbered C6 to C1, C11 to C10, C13 to C11, C5 to C12, C7 to C2, C20 to C3, C2 to C4, C3 to C5, C1 to C6, C19 to C7, C4 to C8, Q1 to Q2, Q2 to Q3, R9 to R1, R1 to R12, R7 to R5, R2 to R6, R5 to R7, U6 to U3, U3 to U4, U4 to U6
Connections:
- net labels added: BATT, BATT_LEVEL, DIFF+, DIFF-, RX_CP+, TX_CP-
- net labels removed: IN1, IN2, RX_CP, TX_CP
- wire segments 146 -> 148
- no-connect marks 36 -> 38
Other:
- note added: "Battery Monitoring"
- moved on the sheet: C4, C6, D2, F1, Q1, R2, R3, R5
